File: hardware/src/PCB/main_pcb.kicad_sch (KiCad schematic)
At the start: 6 parts, among them J3 Hall_effect_sensor, SW2 telemetry_btn, U1 XIAO-nRF52840-Plus-SMD, U4 BME280_sensor, U5 Openlog_SDcard

Commit message: feature: PCB  advancement
Parts:
- removed BZ1: Buzzer_info, Buzzer_Beeper:Buzzer_12x9.5RM7.6, symbol Device:Buzzer
- removed J3: Hall_effect_sensor, Connector_PinHeader_2.54mm:PinHeader_1x03_P2.54mm_Vertical, symbol Connector_Generic:Conn_01x03
- removed SW2: telemetry_btn, craby's_library:SW_BUTT-2, symbol Switch:SW_MEC_5G
- removed U1: XIAO-nRF52840-Plus-SMD, XIAO_Series_Footprints:XIAO-nRF52840-Plus-SMD, symbol Seeed_Studio_XIAO_Series:XIAO-nRF52840_Plus_SMD
- removed U4: BME280_sensor, symbol Enzo's_library:BME_280
- removed U5: Openlog_SDcard, craby's_library:Openlog_SDreader, symbol Enzo's_library:Openlog_SDcard
- added BZ1: Buzzer, Buzzer_Beeper:MagneticBuzzer_ProSignal_ABT-410-RC, symbol main_pcb:Buzzer
- added C1, C3: 2.2 µF - céramique, symbol Device:C_Small
- added C2: 470 µF - électrolytique, symbol Device:C_Small
- added C4: 10 µF - céramique, symbol Device:C_Small
- added C5, C6: 100 nF - céramique, symbol Device:C_Small
- added J1: Pressure_converter, main_pcb:PinHeader_1x03_P2.54mm_Vertical, symbol Connector_Generic:Conn_01x03
- added J2: Hall_sensor, main_pcb:PinHeader_1x03_P2.54mm_Vertical, symbol Connector_Generic:Conn_01x03
- added J3: Pressure_sensor, symbol Connector_Generic:Conn_01x02
- added Q2: BSS84, Package_TO_SOT_SMD:SOT-23, symbol Transistor_FET:BSS84
- added R1, R5: 100 Ω, symbol Device:R
- added R2, R3, R4: 10k Ω, symbol Device:R
- added SW1: Button, Button_Switch_SMD:SW_SPST_B3U-1000P, symbol main_pcb:Button
- added U1: (no value), symbol main_pcb:Aadafruit_12V_booster
- added U2: XIAO-nRF52840-Plus-SMD, main_pcb:XIAO-nRF52840-Plus-SMD, symbol main_pcb:XIAO-nRF52840_Plus_SMD
- added U3: (no value), symbol main_pcb:BME_280
- added U4: (no value), symbol main_pcb:Openlog_SDcard
Connections:
- net +3.3V: now also BZ1.1 (+), C3.2, C6.1, R5.1, U2.12 (3V3)
- net GND: now also BZ1.2 (-), C1.2, C2.2, C3.1, C4.2, C5.2, C6.2, J3.1 (Pin_1), Q2.2 (S), SW1.3 (B), SW1.4 (B), U1.2 (gnd), U2.13 (GND), U2.27 (GND), U2.33 (GND)
- new net: R5.2, U2.3 (P0.28_A2_D2)
- new net: R1.2, U2.1 (P0.02_A0_D0)
- new net +12V: C5.1, J3.2 (Pin_2), Q2.3 (D), U1.3 (Vout)
- new net Button: SW1.1 (A), SW1.2 (A), U2.2 (P0.03_A1_D1)
- new net MOSFET1: Q2.1 (G), R1.1, U1.4 (en_(enable))
- new net VBAT: C1.1, C2.1, C4.1, U1.1 (vcc), U2.32 (VBAT)
- no-connect marks 0 -> 5
Other:
- note added: "Place two 10k homs resistors for the pins SDA and SCL near mcu (because the module is near it)"
- note added: "^{Only for debug}"
- note added: "^{Use to reset place a external button here}"
- title: Cansat_pcb -> Marker_main_pcb

Commit message: feature: PCB advancement
Parts:
- removed Q2: BSS84, Package_TO_SOT_SMD:SOT-23, symbol Transistor_FET:BSS84
- added C7, C8: 100 nF - céramique, symbol Device:C_Small
- added Q1: BSS138, Package_TO_SOT_SMD:SOT-23, symbol Transistor_FET:BSS138
- added R6: 10k Ω, symbol Device:R
Connections:
- net +12V: now also Q1.3 (D)
- net +3.3V: now also J2.1 (Pin_1), R3.1, R4.1, U3.1 (vcc), U3.3 (scl), U3.4 (sda), C7.1, C8.1
- net GND: now also J2.2 (Pin_2), U3.2 (gnd), C7.2, C8.2, Q1.2 (S), R6.2
- net MOSFET1: now also Q1.1 (G), R6.1
- net at J2.3 (Pin_3): now also R2.1
- net SCL1: now reaches R3.2
- net SCL1: now also U2.6 (P0.05_A5_D5_SCL)
- net SDA1: now reaches R4.2
- net SDA1: now also U2.5 (P0.04_A4_D4_SDA)
- net Hall: now reaches R2.2
- net Hall: now also U2.4 (P0.29_A3_D3)
Other:
- note added: "^{Use to reset, place a external btn here}"
- note removed: "Place two 10k homs resistors for the pins SDA and SCL near mcu (because the module is near it)"
- note removed: "^{Use to reset place a external button here}"
- moved on the sheet: C5, J1, J2, J3, R2, R3, R4, U3

Commit message: feature: PCB advancement
Parts:
- added C10, C13: 10 µF - céramique, Capacitor_SMD:C_0603_1608Metric, symbol Device:C_Small
- added C11, C12, C9: 100 nF - céramique, Capacitor_SMD:C_0603_1608Metric, symbol Device:C_Small
- added D1: SS14, Diode_SMD:D_SMA, symbol Diode:SS14
- added Q2, Q3, Q4: BSS138, Package_TO_SOT_SMD:SOT-23, symbol Transistor_FET:BSS138
- added R10, R14, R9: 10k Ω, Resistor_SMD:R_0201_0603Metric, symbol Device:R
- added R11, R12, R13, R8: 100 Ω, Resistor_SMD:R_0201_0603Metric, symbol Device:R
- added R15, R16, R17: 33 Ω, Resistor_SMD:R_0201_0603Metric, symbol Device:R
- added R7: 100k Ω, Resistor_SMD:R_0201_0603Metric, symbol Device:R
- added U5: (no value), symbol main_pcb:Radio_module_CC1101
- C1, C3, C4, C5, C6, C7, C8: footprint (none) -> Capacitor_SMD:C_0603_1608Metric
- C2: footprint (none) -> Capacitor_THT:CP_Radial_D10.0mm_P5.00mm
- J3: footprint (none) -> Connector_PinHeader_1.00mm:PinHeader_1x02_P1.00mm_Vertical
- R1, R2, R3, R4, R5, R6: footprint (none) -> Resistor_SMD:R_0201_0603Metric
Connections:
- net +12V: now also Q1.1 (G), R6.1, R7.1
- net +3.3V: now also J2.3 (Pin_3), R2.1, U4.4 (vcc), C10.1, C12.2, C13.2, C9.1, Q2.3 (D), Q3.3 (D), Q4.3 (D), U5.2 (VCC); no longer R3.1, R4.1, U3.3 (scl), U3.4 (sda)
- net Button: now also U2.1 (P0.02_A0_D0); no longer U2.2 (P0.03_A1_D1)
- net GND: now also U4.5 (gnd), C10.2, C11.2, C12.1, C13.1, C9.2, Q2.2 (S), Q3.2 (S), Q4.2 (S), R10.2, R14.2, R9.2, U5.1 (GND)
- net MOSFET1: now also R7.2; no longer Q1.1 (G), R6.1, U1.4 (en_(enable))
- net SCL1: now also U3.3 (scl); no longer R3.2
- net SDA1: now also U3.4 (sda); no longer R4.2
- net VBAT: now also C11.1, D1.2 (A); no longer C1.1, C2.1, U2.32 (VBAT)
- net SD_RX: now reaches U4.2 (rxi)
- net SD_RX: now also R12.1
- net SD_TX: now reaches U4.3 (txo)
- net SD_TX: now also R13.1
- net at R5.2: now also U2.2 (P0.03_A1_D1); no longer U2.3 (P0.28_A2_D2)
- net at R1.2: now also U2.15 (P0.15_D11_I2S_SD); no longer U2.1 (P0.02_A0_D0)
- net at U2.16 (P0.19_D12_I2S_SCK): now also R8.2
- net at U2.17 (P1.01_D13_I2S_WS): now also R11.2
- net at U2.20 (P0.31_D16_BAT): now also C1.1, C2.1, U2.32 (VBAT), D1.1 (K)
- net at U2.21 (P1.03_D17_SCK1): now also R15.2
- net at U2.22 (P1.05_D18_MISO1): now also R16.2
- net at U2.23 (P1.07_D19_MOSI1): now also R17.2
- net Rst_btn: now reaches U2.26 (REST)
- net at U2.7 (P1.11_D6_TX): now also R12.2
- net at U2.8 (P1.12_D7_RX): now also R13.2
- new net MISO1: R16.1
- new net MOSFET2: Q2.1 (G), Q4.1 (G), R14.1, R8.1, R9.1
- new net MOSFET3: Q3.1 (G), R10.1, R11.1
- new net MOSI1: R17.1
- new net SCK1: R15.1
- no-connect marks 5 -> 8
Other:
- note added: "^{Cutting power module function}"
- note added: "^{Need to see if we had the pull resistor on the two pins in the real module there are already place it in the scl and sda but need to confirm}"
- note removed: "^{Use to reset, place a external btn here}"
- moved on the sheet: BZ1, C2, C4, C6, C7, C8, J1, J2, R1, R2, R3, R4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

Commit message: feature: PCB advancement
Parts:
- removed J1: Pressure_converter, main_pcb:PinHeader_1x03_P2.54mm_Vertical, symbol Connector_Generic:Conn_01x03
- removed Q4: BSS138, Package_TO_SOT_SMD:SOT-23, symbol Transistor_FET:BSS138
- removed R14: 10k Ω, Resistor_SMD:R_0201_0603Metric, symbol Device:R
- added J1: Batt, PCM_SparkFun-Connector:JST_1x02_P2.0mm_Horizontal_SMD, symbol Connector_Generic:Conn_01x02
- added SW2: Button, Button_Switch_SMD:SW_SPST_B3U-1000P, symbol main_pcb:Button
Connections:
- net +12V: now also U1.4 (en_(enable))
- net GND: now also J1.2 (Pin_2), SW2.3 (B), SW2.4 (B); no longer U2.27 (GND)
- net MISO1: now also U2.10 (P1.14_D9_MISO), U5.7 (MISO); no longer R16.1
- net MOSI1: now also U5.6 (MOSI)
- net Rst_btn: now also SW2.1 (A), SW2.2 (A)
- net SCK1: now also U5.5 (SCK)
- net VBAT: now also J1.1 (Pin_1)
- net at R16.2: now also U2.21 (P1.03_D17_SCK1); no longer U2.22 (P1.05_D18_MISO1)
- net at R17.2: now also U2.9 (P1.13_D8_SCK); no longer U2.23 (P1.07_D19_MOSI1)
- net at R15.2: now also U2.11 (P1.15_D10_MOSI); no longer U2.21 (P1.03_D17_SCK1)
- net RF_GDO0: now reaches U5.3 (GDO0)
- net RF_GDO0: now also U2.23 (P1.07_D19_MOSI1)
- net RF_CSN: now reaches U5.4 (CSN)
- net RF_CSN: now also R16.1
- no-connect marks 8 -> 10
Other:
- note added: "^{SD card writer}"
- moved on the sheet: C10, C11, C12, C13, C4, C5, C7, C8, C9, J2, J3, Q1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

Commit message: feature: PCB advancement
Parts:
- removed Q1, Q3: BSS138, Package_TO_SOT_SMD:SOT-23, symbol Transistor_FET:BSS138
- removed R6, R9: 10k Ω, Resistor_SMD:R_0201_0603Metric, symbol Device:R
- added C14: 10 µF - céramique, Capacitor_SMD:C_0603_1608Metric, symbol Device:C_Small
- added Q1, Q3, Q4: BSS84, Package_TO_SOT_SMD:SOT-23, symbol Transistor_FET:BSS84
- added R14, R18, R19, R20: 100k Ω, Resistor_SMD:R_0201_0603Metric, symbol Device:R
- R10: value 10k Ω -> 100k Ω
Connections:
- net MOSFET1 is gone; now on net GND: R1.1, R7.2
- net VBAT is gone; now on net +3.3V: C11.1, C4.1, D1.2 (A), J1.1 (Pin_1), U1.1 (vcc)
- net +12V: now also C14.2, Q4.2 (S), Q4.3 (D), R18.2; no longer R7.1, U1.4 (en_(enable))
- net +3.3V: now also R10.2, Q1.2 (S), Q1.3 (D), Q3.2 (S), Q3.3 (D), R14.2; no longer Q2.3 (D)
- net GND: now also Q2.1 (G), C14.1, R19.1, R19.2; no longer R10.2
- net MOSFET2: now also Q3.1 (G), R14.1; no longer Q2.1 (G)
- net MOSFET3: now also Q1.1 (G)
- new net: R7.1, U1.4 (en_(enable))
- new net: Q2.3 (D), R20.2
- new net: Q4.1 (G), R18.1, R20.1
Other:
- note added: "Need to see if we had the pull resistor on the two pins in the real module there are already place it in the scl and sda but need to confirm"
- note added: "^{Cutting power module function for hall_sensor}"
- note added: "^{Cutting power module function for openlog}"
- note added: "^{Cutting power module function for water_sensor}"
- note removed: "^{Cutting power module function}"
- note removed: "^{Need to see if we had the pull resistor on the two pins in the real module there are already place it in the scl and sda but need to confirm}"
- moved on the sheet: C10, C11, C12, C13, C4, C5, C7, C9, J1, J3, R10, R3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

Commit message: feature: PCB advancement
Parts:
- added C15, C16: 100 nF - céramique, Capacitor_SMD:C_0603_1608Metric, symbol Device:C_Small
- added D2: 1N4148W, Diode_SMD:D_SOD-123, symbol Diode:1N4148W
- added R6: 1k Ω, Resistor_SMD:R_0201_0603Metric, symbol Device:R
- added U6: (no value), main_pcb:DFrobot, symbol main_pcb:DFrobot
Connections:
- net +12V: now also U6.1 (I+), U6.2 (I-)
- net +3.3V: now also C15.2, D2.2 (A), U6.4 (VCC)
- net GND: now also C15.1, C16.2, D2.1 (K), U6.3 (GND)
- net at U2.3 (P0.28_A2_D2): now also C16.1, R6.2
- new net PressureA: R6.1, U6.5 (A(sig))
Other:
- moved on the sheet: C6

Commit message: feature: PCB advancement
Parts:
- J3: footprint Connector_PinHeader_1.00mm:PinHeader_1x02_P1.00mm_Vertical -> Connector_PinHeader_2.54mm:PinHeader_1x02_P2.54mm_Vertical
- U1: footprint (none) -> main_pcb:Adafruit_TPS61040_5644
- U3: footprint (none) -> main_pcb:BME280
- U4: footprint (none) -> main_pcb:OpenLog
Other:
- moved on the sheet: C5, C7
Changed lines of the file:
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@@
 	)
 	(junction
-		(at 195.58 53.34)
+		(at 256.54 44.45)
 		(diameter 0)
 		(color 0 0 0 0)
 	)
 	(junction
-		(at 256.54 44.45)
+		(at 195.58 53.34)
 		(diameter 0)
 		(color 0 0 0 0)
 	)
 	(junction
-		(at 96.52 34.29)
+		(at 100.33 34.29)
 		(diameter 0)
 		(color 0 0 0 0)
@@
 	)
 	(junction
-		(at 48.26 62.23)
+		(at 45.72 63.5)
 		(diameter 0)
 		(color 0 0 0 0)
 	)
 	(junction
-		(at 46.99 69.85)
+		(at 44.45 71.12)
 		(diameter 0)
 		(color 0 0 0 0)
@@
 	)
 	(junction
-		(at 96.52 39.37)
+		(at 100.33 39.37)
 		(diameter 0)
 		(color 0 0 0 0)
@@
 	)
 	(junction
-		(at 46.99 62.23)
+		(at 44.45 63.5)
 		(diameter 0)
 		(color 0 0 0 0)
@@
 	(wire
 		(pts
-			(xy 43.18 66.04) (xy 43.18 62.23)
+			(xy 43.18 66.04) (xy 43.18 63.5)
 		)
 		(stroke
@@
 	(wire
 		(pts
-			(xy 46.99 62.23) (xy 46.99 63.5)
+			(xy 44.45 63.5) (xy 44.45 64.77)
 		)
 		(stroke
@@
 	(wire
 		(pts
-			(xy 96.52 40.64) (xy 96.52 39.37)
+			(xy 100.33 40.64) (xy 100.33 39.37)
 		)
 		(stroke
@@
 	(wire
 		(pts
-			(xy 99.06 35.56) (xy 99.06 34.29)
+			(xy 102.87 35.56) (xy 102.87 34.29)
 		)
 		(stroke
@@
 	(wire
 		(pts
-			(xy 99.06 35.56) (xy 104.14 35.56)
+			(xy 102.87 35.56) (xy 104.14 35.56)
 		)
 		(stroke
@@
 	(wire
 		(pts
-			(xy 46.99 68.58) (xy 46.99 69.85)
+			(xy 44.45 69.85) (xy 44.45 71.12)
 		)
 		(stroke
@@
 	(wire
 		(pts
-			(xy 46.99 62.23) (xy 48.26 62.23)
+			(xy 44.45 63.5) (xy 45.72 63.5)
 		)
 		(stroke
@@
 	(wire
 		(pts
-			(xy 99.06 38.1) (xy 104.14 38.1)
+			(xy 102.87 38.1) (xy 104.14 38.1)
 		)
 		(stroke
@@
 	(wire
 		(pts
-			(xy 48.26 62.23) (xy 49.53 62.23)
+			(xy 45.72 63.5) (xy 46.99 63.5)
 		)
 		(stroke
@@
 	(wire
 		(pts
-			(xy 96.52 39.37) (xy 99.06 39.37)
+			(xy 100.33 39.37) (xy 102.87 39.37)
 		)
 		(stroke
@@
 	(wire
 		(pts
-			(xy 43.18 69.85) (xy 46.99 69.85)
+			(xy 43.18 71.12) (xy 44.45 71.12)
 		)
 		(stroke
@@
 	(wire
 		(pts
-			(xy 48.26 60.96) (xy 48.26 62.23)
+			(xy 45.72 62.23) (xy 45.72 63.5)
 		)
 		(stroke
@@
 	(wire
 		(pts
-			(xy 43.18 68.58) (xy 43.18 69.85)
+			(xy 43.18 68.58) (xy 43.18 71.12)
 		)
 		(stroke
@@
 	(wire
 		(pts
-			(xy 46.99 69.85) (xy 46.99 71.12)
+			(xy 44.45 71.12) (xy 44.45 72.39)
 		)
 		(stroke
@@
 	(wire
 		(pts
-			(xy 43.18 62.23) (xy 46.99 62.23)
+			(xy 43.18 63.5) (xy 44.45 63.5)
 		)
 		(stroke
@@
 	(wire
 		(pts
-			(xy 96.52 34.29) (xy 99.06 34.29)
+			(xy 100.33 34.29) (xy 102.87 34.29)
 		)
 		(stroke
@@
 	(wire
 		(pts
-			(xy 99.06 39.37) (xy 99.06 38.1)
+			(xy 102.87 39.37) (xy 102.87 38.1)
 		)
 		(stroke
@@
 	(wire
 		(pts
-			(xy 96.52 33.02) (xy 96.52 34.29)
+			(xy 100.33 33.02) (xy 100.33 34.29)
 		)
 		(stroke
@@
 	(hierarchical_label "Pressure-"
 		(shape input)
-		(at 49.53 62.23 0)
+		(at 46.99 63.5 0)
 		(effects
 			(font
@@
 			)
 		)
-		(property "Footprint" ""
+		(property "Footprint" "main_pcb:OpenLog"
 			(at 201.93 55.88 0)
 			(hide yes)
@@
 			)
 		)
-		(property "Footprint" ""
+		(property "Footprint" "main_pcb:BME280"
 			(at 106.68 44.45 0)
 			(hide yes)
@@
 	(symbol
 		(lib_id "power:+12V")
-		(at 48.26 60.96 0)
+		(at 45.72 62.23 0)
 		(unit 1)
 		(body_style 1)
@@
 		(dnp no)
 		(property "Reference" "#PWR03"
-			(at 48.26 64.77 0)
+			(at 45.72 66.04 0)
 			(hide yes)
 			(show_name no)
@@
 		)
 		(property "Value" "+12V"
-			(at 48.006 57.15 0)
+			(at 45.466 58.42 0)
 			(show_name no)
 			(do_not_autoplace no)
@@
 		)
 		(property "Footprint" ""
-			(at 48.26 60.96 0)
+			(at 45.72 62.23 0)
 			(hide yes)
 			(show_name no)
@@
 		)
 		(property "Datasheet" ""
-			(at 48.26 60.96 0)
+			(at 45.72 62.23 0)
 			(hide yes)
 			(show_name no)
@@
 		)
 		(property "Description" "Power symbol creates a global label with name \"+12V\""
-			(at 48.26 60.96 0)
+			(at 45.72 62.23 0)
 			(hide yes)
 			(show_name no)
@@
 	(symbol
 		(lib_id "Device:C_Small")
-		(at 46.99 66.04 0)
+		(at 44.45 67.31 0)
 		(unit 1)
 		(body_style 1)
@@
 		(dnp no)
 		(property "Reference" "C5"
-			(at 48.768 66.04 0)
+			(at 46.228 67.31 0)
 			(show_name no)
 			(do_not_autoplace no)
@@
 		)
 		(property "Value" "100 nF - céramique"
-			(at 47.498 68.072 0)
+			(at 44.958 69.342 0)
 			(show_name no)
 			(do_not_autoplace no)
@@
 		)
 		(property "Footprint" "Capacitor_SMD:C_0603_1608Metric"
-			(at 46.99 66.04 0)
+			(at 44.45 67.31 0)
 			(hide yes)
 			(show_name no)
@@
 		)
 		(property "Datasheet" ""
-			(at 46.99 66.04 0)
+			(at 44.45 67.31 0)
 			(hide yes)
 			(show_name no)
@@
 		)
 		(property "Description" "Unpolarized capacitor, small symbol"
-			(at 46.99 66.04 0)
+			(at 44.45 67.31 0)
 			(hide yes)
 			(show_name no)
@@
 	(symbol
 		(lib_id "power:Earth")
-		(at 46.99 71.12 0)
+		(at 44.45 72.39 0)
 		(unit 1)
 		(body_style 1)
@@
 		(dnp no)
 		(property "Reference" "#PWR012"
-			(at 46.99 77.47 0)
+			(at 44.45 78.74 0)
 			(hide yes)
 			(show_name no)
@@
 		)
 		(property "Value" "GND"
-			(at 46.99 74.93 0)
+			(at 44.45 76.2 0)
 			(show_name no)
 			(do_not_autoplace no)
@@
 		)
 		(property "Footprint" ""
-			(at 46.99 71.12 0)
+			(at 44.45 72.39 0)
 			(hide yes)
 			(show_name no)
@@
 		)
 		(property "Datasheet" ""
-			(at 46.99 71.12 0)
+			(at 44.45 72.39 0)
 			(hide yes)
 			(show_name no)
@@
 		)
 		(property "Description" "Power symbol creates a global label with name \"Earth\""
-			(at 46.99 71.12 0)
+			(at 44.45 72.39 0)
 			(hide yes)
 			(show_name no)
@@
 	(symbol
 		(lib_id "power:Earth")
-		(at 96.52 40.64 0)
+		(at 100.33 40.64 0)
 		(unit 1)
 		(body_style 1)
@@
 		(dnp no)
 		(property "Reference" "#PWR011"
-			(at 96.52 46.99 0)
+			(at 100.33 46.99 0)
 			(hide yes)
 			(show_name no)
@@
 		)
 		(property "Value" "GND"
-			(at 96.52 44.45 0)
+			(at 100.33 44.45 0)
 			(show_name no)
 			(do_not_autoplace no)
@@
 		)
 		(property "Footprint" ""
-			(at 96.52 40.64 0)
+			(at 100.33 40.64 0)
 			(hide yes)
 			(show_name no)
@@
 		)
 		(property "Datasheet" ""
-			(at 96.52 40.64 0)
+			(at 100.33 40.64 0)
 			(hide yes)
 			(show_name no)
@@
 		)
 		(property "Description" "Power symbol creates a global label with name \"Earth\""
-			(at 96.52 40.64 0)
+			(at 100.33 40.64 0)
 			(hide yes)
 			(show_name no)
@@
 	(symbol
 		(lib_id "Device:C_Small")
-		(at 96.52 36.83 0)
+		(at 100.33 36.83 0)
 		(unit 1)
 		(body_style 1)
@@
 		(dnp no)
 		(property "Reference" "C7"
-			(at 91.694 36.83 0)
+			(at 95.504 36.83 0)
 			(show_name no)
 			(do_not_autoplace no)
@@
 		)
 		(property "Value" "100 nF - céramique"
-			(at 75.184 39.116 0)
+			(at 78.994 39.116 0)
 			(show_name no)
 			(do_not_autoplace no)
@@
 		)
 		(property "Footprint" "Capacitor_SMD:C_0603_1608Metric"
-			(at 96.52 36.83 0)
+			(at 100.33 36.83 0)
 			(hide yes)
 			(show_name no)
@@
 		)
 		(property "Datasheet" ""
-			(at 96.52 36.83 0)
+			(at 100.33 36.83 0)
 			(hide yes)
 			(show_name no)
@@
 		)
 		(property "Description" "Unpolarized capacitor, small symbol"
-			(at 96.52 36.83 0)
+			(at 100.33 36.83 0)
 			(hide yes)
 			(show_name no)
@@
 	(symbol
 		(lib_id "power:+3.3V")
-		(at 96.52 33.02 0)
+		(at 100.33 33.02 0)
 		(mirror y)
 		(unit 1)
@@
 		(dnp no)
 		(property "Reference" "#PWR020"
-			(at 96.52 36.83 0)
+			(at 100.33 36.83 0)
 			(hide yes)
 			(show_name no)
@@
 		)
 		(property "Value" "+3.3V"
-			(at 98.806 29.464 0)
+			(at 102.616 29.464 0)
 			(show_name no)
 			(do_not_autoplace no)
@@
 		)
 		(property "Footprint" ""
-			(at 96.52 33.02 0)
+			(at 100.33 33.02 0)
 			(hide yes)
 			(show_name no)
@@
 		)
 		(property "Datasheet" ""
-			(at 96.52 33.02 0)
+			(at 100.33 33.02 0)
 			(hide yes)
 			(show_name no)
@@
 		)
 		(property "Description" "Power symbol creates a global label with name \"+3.3V\""
-			(at 96.52 33.02 0)
+			(at 100.33 33.02 0)
 			(hide yes)
 			(show_name no)
@@
 			)
 		)
-		(property "Footprint" "Connector_PinHeader_1.00mm:PinHeader_1x02_P1.00mm_Vertical"
+		(property "Footprint" "Connector_PinHeader_2.54mm:PinHeader_1x02_P2.54mm_Vertical"
 			(at 38.1 68.58 0)
 			(hide yes)
@@
 			)
 		)
-		(property "Footprint" ""
+		(property "Footprint" "main_pcb:Adafruit_TPS61040_5644"
 			(at 102.87 127 0)
 			(hide yes)

Commit message: feature: PCB advancement
Parts:
- removed C1: 2.2 µF - céramique, Capacitor_SMD:C_0603_1608Metric, symbol Device:C_Small
- removed Q1, Q3: BSS84, Package_TO_SOT_SMD:SOT-23, symbol Transistor_FET:BSS84
- added C17: 220 µF - électrolytique, Capacitor_THT:CP_Radial_D10.0mm_P5.00mm, symbol Device:C_Small
- added Q5, Q6: IRF9530, main_pcb:TRANS_IRF9530, symbol Transistor_FET:BSS84
- C2: value 470 µF - électrolytique -> 47 µF - électrolytique
- D1: value SS14 -> 1N5819
- D2: value 1N4148W -> fr107
- Q2: value BSS138 -> BS170; footprint Package_TO_SOT_SMD:SOT-23 -> main_pcb:TO92
- Q4: value BSS84 -> IRF9530; footprint Package_TO_SOT_SMD:SOT-23 -> main_pcb:TRANS_IRF9530
- R15, R16: footprint Resistor_SMD:R_0201_0603Metric -> main_pcb:R_1206_3216Metric
Connections:
- net +3.3V: now also C17.1, Q5.2 (S), Q5.3 (D), Q6.2 (S), Q6.3 (D)
- net GND: now also C17.2
- net MOSFET2: now also Q5.1 (G)
- net MOSFET3: now also Q6.1 (G)
Other:
- moved on the sheet: D1
