File: hardware/src/PCB/main_pcb.kicad_sch (KiCad schematic)
At the start: 53 parts, among them J1 Batt, J2 Hall_sensor, J3 Pressure_sensor, Q2 BS170, Q4 IRF9530, Q5 IRF9530, Q6 IRF9530, SW1 Button, SW2 Button, U2 XIAO-nRF52840-Plus-SMD

Commit message: feature: PCB advancement
Parts:
- D1: footprint Diode_SMD:D_SMA -> main_pcb:DIOAD1036W78L470D235
- D2: footprint Diode_SMD:D_SOD-123 -> main_pcb:DIOAD1036W78L470D235
- J1: footprint PCM_SparkFun-Connector:JST_1x02_P2.0mm_Horizontal_SMD -> Connector_PinHeader_1.00mm:PinHeader_1x02_P1.00mm_Horizontal
- R1, R10, R11, R12, R13, R14, R17, R18, R19, R2, R20, R3, R4, R5, R6, R7, R8: footprint Resistor_SMD:R_0201_0603Metric -> main_pcb:R_1206_3216Metric
Changed lines of the file:
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@@
 			)
 		)
-		(property "Footprint" "Resistor_SMD:R_0201_0603Metric"
+		(property "Footprint" "main_pcb:R_1206_3216Metric"
 			(at 96.012 132.08 90)
 			(hide yes)
@@
 			)
 		)
-		(property "Footprint" "Resistor_SMD:R_0201_0603Metric"
+		(property "Footprint" "main_pcb:R_1206_3216Metric"
 			(at 198.12 144.018 90)
 			(hide yes)
@@
 			)
 		)
-		(property "Footprint" "Resistor_SMD:R_0201_0603Metric"
+		(property "Footprint" "main_pcb:R_1206_3216Metric"
 			(at 99.822 57.15 90)
 			(hide yes)
@@
 			)
 		)
-		(property "Footprint" "Resistor_SMD:R_0201_0603Metric"
+		(property "Footprint" "main_pcb:R_1206_3216Metric"
 			(at 116.84 160.782 90)
 			(hide yes)
@@
 			)
 		)
-		(property "Footprint" "Diode_SMD:D_SOD-123"
+		(property "Footprint" "main_pcb:DIOAD1036W78L470D235"
 			(at 228.6 89.535 0)
 			(hide yes)
@@
 			)
 		)
-		(property "Footprint" "Resistor_SMD:R_0201_0603Metric"
+		(property "Footprint" "main_pcb:R_1206_3216Metric"
 			(at 198.12 132.588 90)
 			(hide yes)
@@
 			)
 		)
-		(property "Footprint" "Resistor_SMD:R_0201_0603Metric"
+		(property "Footprint" "main_pcb:R_1206_3216Metric"
 			(at 66.802 170.18 90)
 			(hide yes)
@@
 			)
 		)
-		(property "Footprint" "Resistor_SMD:R_0201_0603Metric"
+		(property "Footprint" "main_pcb:R_1206_3216Metric"
 			(at 256.54 129.032 90)
 			(hide yes)
@@
 			)
 		)
-		(property "Footprint" "Resistor_SMD:R_0201_0603Metric"
+		(property "Footprint" "main_pcb:R_1206_3216Metric"
 			(at 180.34 117.348 90)
 			(hide yes)
@@
 			)
 		)
-		(property "Footprint" "Diode_SMD:D_SMA"
+		(property "Footprint" "main_pcb:DIOAD1036W78L470D235"
 			(at 193.04 155.575 0)
 			(hide yes)
@@
 			)
 		)
-		(property "Footprint" "PCM_SparkFun-Connector:JST_1x02_P2.0mm_Horizontal_SMD"
+		(property "Footprint" "Connector_PinHeader_1.00mm:PinHeader_1x02_P1.00mm_Horizontal"
 			(at 39.37 123.19 0)
 			(hide yes)
@@
 			)
 		)
-		(property "Footprint" "Resistor_SMD:R_0201_0603Metric"
+		(property "Footprint" "main_pcb:R_1206_3216Metric"
 			(at 102.362 58.42 90)
 			(hide yes)
@@
 			)
 		)
-		(property "Footprint" "Resistor_SMD:R_0201_0603Metric"
+		(property "Footprint" "main_pcb:R_1206_3216Metric"
 			(at 120.142 170.18 90)
 			(hide yes)
@@
 			)
 		)
-		(property "Footprint" "Resistor_SMD:R_0201_0603Metric"
+		(property "Footprint" "main_pcb:R_1206_3216Metric"
 			(at 198.12 113.538 90)
 			(hide yes)
@@
 			)
 		)
-		(property "Footprint" "Resistor_SMD:R_0201_0603Metric"
+		(property "Footprint" "main_pcb:R_1206_3216Metric"
 			(at 256.54 125.222 90)
 			(hide yes)
@@
 			)
 		)
-		(property "Footprint" "Resistor_SMD:R_0201_0603Metric"
+		(property "Footprint" "main_pcb:R_1206_3216Metric"
 			(at 31.242 170.18 90)
 			(hide yes)
@@
 			)
 		)
-		(property "Footprint" "Resistor_SMD:R_0201_0603Metric"
+		(property "Footprint" "main_pcb:R_1206_3216Metric"
 			(at 46.482 44.45 90)
 			(hide yes)
@@
 			)
 		)
-		(property "Footprint" "Resistor_SMD:R_0201_0603Metric"
+		(property "Footprint" "main_pcb:R_1206_3216Metric"
 			(at 198.12 136.398 90)
 			(hide yes)
@@
 			)
 		)
-		(property "Footprint" "Resistor_SMD:R_0201_0603Metric"
+		(property "Footprint" "main_pcb:R_1206_3216Metric"
 			(at 98.552 170.18 90)
 			(hide yes)
@@
 			)
 		)
-		(property "Footprint" "Resistor_SMD:R_0201_0603Metric"
+		(property "Footprint" "main_pcb:R_1206_3216Metric"
 			(at 198.12 140.208 90)
 			(hide yes)

Commit message: feature: PCB advancement
Parts:
- removed C16: 100 nF - céramique, Capacitor_SMD:C_0603_1608Metric, symbol Device:C_Small
- J1: footprint Connector_PinHeader_1.00mm:PinHeader_1x02_P1.00mm_Horizontal -> Connector_PinHeader_2.54mm:PinHeader_1x02_P2.54mm_Horizontal
Connections:
- net GND: now also Q2.3 (D); no longer Q2.2 (S)
- net at R20.2: now also Q2.2 (S); no longer Q2.3 (D)
Other:
- moved on the sheet: R6
Changed lines of the file:
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@@
 	)
 	(junction
-		(at 185.42 115.57)
-		(diameter 0)
-		(color 0 0 0 0)
-	)
-	(junction
 		(at 95.25 127)
 		(diameter 0)
@@
 	(wire
 		(pts
-			(xy 184.15 120.65) (xy 185.42 120.65)
-		)
-		(stroke
-			(width 0)
-			(type default)
-		)
-	)
-	(wire
-		(pts
 			(xy 224.79 83.82) (xy 224.79 85.09)
 		)
@@
 	(wire
 		(pts
-			(xy 185.42 115.57) (xy 203.2 115.57)
-		)
-		(stroke
-			(width 0)
-			(type default)
-		)
-	)
-	(wire
-		(pts
 			(xy 251.46 115.57) (xy 252.73 115.57)
 		)
@@
 	(wire
 		(pts
-			(xy 175.26 115.57) (xy 176.53 115.57)
+			(xy 193.04 115.57) (xy 194.31 115.57)
 		)
 		(stroke
@@
 	(wire
 		(pts
-			(xy 184.15 115.57) (xy 185.42 115.57)
+			(xy 201.93 115.57) (xy 203.2 115.57)
 		)
 		(stroke
@@
 	(hierarchical_label "PressureA"
 		(shape input)
-		(at 175.26 115.57 180)
+		(at 193.04 115.57 180)
 		(effects
 			(font
@@
 		(lib_id "Transistor_FET:BSS138")
 		(at 106.68 165.1 0)
+		(mirror x)
 		(unit 1)
 		(body_style 1)
@@
 		)
 		(property "Footprint" "main_pcb:TO92"
-			(at 111.76 167.005 0)
+			(at 111.76 163.195 0)
 			(hide yes)
 			(show_name no)
@@
 		)
 		(property "Datasheet" "https://www.onsemi.com/pub/Collateral/BSS138-D.PDF"
-			(at 111.76 168.91 0)
+			(at 111.76 161.29 0)
 			(hide yes)
 			(show_name no)
@@
 	(symbol
 		(lib_id "Device:R")
-		(at 180.34 115.57 90)
+		(at 198.12 115.57 90)
 		(unit 1)
 		(body_style 1)
@@
 		(dnp no)
 		(property "Reference" "R6"
-			(at 180.34 115.57 90)
+			(at 198.12 115.57 90)
 			(show_name no)
 			(do_not_autoplace no)
@@
 		)
 		(property "Value" "1k Ω"
-			(at 180.086 113.538 90)
+			(at 197.866 117.602 90)
 			(show_name no)
 			(do_not_autoplace no)
@@
 		)
 		(property "Footprint" "main_pcb:R_1206_3216Metric"
-			(at 180.34 117.348 90)
+			(at 198.12 117.348 90)
 			(hide yes)
 			(show_name no)
@@
 		)
 		(property "Datasheet" ""
-			(at 180.34 115.57 0)
+			(at 198.12 115.57 0)
 			(hide yes)
 			(show_name no)
@@
 		)
 		(property "Description" "Resistor"
-			(at 180.34 115.57 0)
+			(at 198.12 115.57 0)
 			(hide yes)
 			(show_name no)
@@
 			)
 		)
-		(property "Footprint" "Connector_PinHeader_1.00mm:PinHeader_1x02_P1.00mm_Horizontal"
+		(property "Footprint" "Connector_PinHeader_2.54mm:PinHeader_1x02_P2.54mm_Horizontal"
 			(at 39.37 123.19 0)
 			(hide yes)
@@
 	)
 	(symbol
-		(lib_id "power:Earth")
-		(at 184.15 120.65 270)
-		(unit 1)
-		(body_style 1)
-		(exclude_from_sim no)
-		(in_bom yes)
-		(on_board yes)
-		(in_pos_files yes)
-		(dnp no)
-		(property "Reference" "#PWR033"
-			(at 177.8 120.65 0)
-			(hide yes)
-			(show_name no)
-			(do_not_autoplace no)
-			(effects
-				(font
-					(size 1.27 1.27)
-				)
-			)
-		)
-		(property "Value" "GND"
-			(at 179.324 120.65 90)
-			(show_name no)
-			(do_not_autoplace no)
-			(effects
-				(font
-					(size 1.1684 1.1684)
-				)
-			)
-		)
-		(property "Footprint" ""
-			(at 184.15 120.65 0)
-			(hide yes)
-			(show_name no)
-			(do_not_autoplace no)
-			(effects
-				(font
-					(size 1.27 1.27)
-				)
-			)
-		)
-		(property "Datasheet" ""
-			(at 184.15 120.65 0)
-			(hide yes)
-			(show_name no)
-			(do_not_autoplace no)
-			(effects
-				(font
-					(size 1.27 1.27)
-				)
-			)
-		)
-		(property "Description" "Power symbol creates a global label with name \"Earth\""
-			(at 184.15 120.65 0)
-			(hide yes)
-			(show_name no)
-			(do_not_autoplace no)
-			(effects
-				(font
-					(size 1.27 1.27)
-				)
-			)
-		)
-		(pin "1"
-		)
-		(instances
-			(project "main_pcb"
-				(path "/f7c433f5-979d-4748-9c6b-df3b09da91ad"
-					(reference "#PWR033")
-					(unit 1)
-				)
-			)
-		)
-	)
-	(symbol
 		(lib_id "Device:R")
 		(at 104.14 58.42 0)
@@
 					(unit 1)
 				)
-			)
-		)
-	)
-	(symbol
-		(lib_id "Device:C_Small")
-		(at 185.42 118.11 0)
-		(unit 1)
-		(body_style 1)
-		(exclude_from_sim no)
-		(in_bom yes)
-		(on_board yes)
-		(in_pos_files yes)
-		(dnp no)
-		(property "Reference" "C16"
-			(at 183.642 114.3 0)
-			(show_name no)
-			(do_not_autoplace no)
-			(effects
-				(font
-					(size 1.27 1.27)
-				)
-				(justify left)
-			)
-		)
-		(property "Value" "100 nF - céramique"
-			(at 176.276 104.902 0)
-			(show_name no)
-			(do_not_autoplace no)
-			(effects
-				(font
-					(size 1.27 1.27)
-				)
-				(justify left)
-			)
-		)
-		(property "Footprint" "Capacitor_SMD:C_0603_1608Metric"
-			(at 185.42 118.11 0)
-			(hide yes)
-			(show_name no)
-			(do_not_autoplace no)
-			(effects
-				(font
-					(size 1.27 1.27)
-				)
-			)
-		)
-		(property "Datasheet" ""
-			(at 185.42 118.11 0)
-			(hide yes)
-			(show_name no)
-			(do_not_autoplace no)
-			(effects
-				(font
-					(size 1.27 1.27)
-				)
-			)
-		)
-		(property "Description" "Unpolarized capacitor, small symbol"
-			(at 185.42 118.11 0)
-			(hide yes)
-			(show_name no)
-			(do_not_autoplace no)
-			(effects
-				(font
-					(size 1.27 1.27)
-				)
-			)
-		)
-		(pin "2"
-		)
-		(pin "1"
-		)
-		(instances
-			(project "main_pcb"
-				(path "/f7c433f5-979d-4748-9c6b-df3b09da91ad"
-					(reference "C16")
-					(unit 1)
-				)

Commit message: feature: PCB advancement
Parts:
- removed C10, C13, C14, C4: 10 µF - céramique, Capacitor_SMD:C_0603_1608Metric, symbol Device:C_Small
- removed R20: 100k Ω, main_pcb:R_1206_3216Metric, symbol Device:R
- removed R3, R4: 10k Ω, main_pcb:R_1206_3216Metric, symbol Device:R
- C17: footprint Capacitor_THT:CP_Radial_D10.0mm_P5.00mm -> Capacitor_THT:CP_Radial_D8.0mm_P3.50mm
- J1: footprint Connector_PinHeader_2.54mm:PinHeader_1x02_P2.54mm_Horizontal -> Connector_PinHeader_2.54mm:PinHeader_1x02_P2.54mm_Vertical
Connections:
- net +12V: no longer Q4.2 (S), Q4.3 (D), R18.2
- net +3.3V: now also Q4.2 (S), R18.2; no longer C11.1, U1.1 (vcc)
- net at Q2.2 (S): now also Q4.1 (G), R18.1
- new net Transistor+: C11.1, Q4.3 (D), U1.1 (vcc)
Other:
- note removed: "Need to see if we had the pull resistor on the two pins in the real module there are already place it in the scl and sda but need to confirm"
- moved on the sheet: C11, C15, C9, Q2, R19, R7, U6

Commit message: feature: PCB advancement
Parts:
- removed U6: (no value), main_pcb:DFrobot, symbol main_pcb:DFrobot
- added J4: Pressure_pins, Connector_PinHeader_2.54mm:PinHeader_1x02_P2.54mm_Vertical, symbol Connector_Generic:Conn_01x02
- added J5: converter_pins, main_pcb:PinHeader_1x03_P2.54mm_Vertical, symbol Connector_Generic:Conn_01x03
Connections:
- net +12V: now also J4.1 (Pin_1), J4.2 (Pin_2)
- net +3.3V: now also J5.2 (Pin_2)
- net GND: now also J5.1 (Pin_1)
- net PressureA: now also J5.3 (Pin_3)
Changed lines of the file:
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@@
 	)
 	(symbol
-		(lib_id "main_pcb:DFrobot")
-		(at 93.98 72.39 0)
-		(unit 1)
-		(body_style 1)
-		(exclude_from_sim no)
-		(in_bom yes)
-		(on_board yes)
-		(in_pos_files yes)
-		(dnp no)
-		(property "Reference" "U6"
-			(at 101.854 63.754 0)
-			(show_name no)
-			(do_not_autoplace no)
-			(effects
-				(font
-					(size 1.27 1.27)
-				)
-			)
-		)
-		(property "Value" ""
-			(at 93.98 72.39 0)
-			(show_name no)
-			(do_not_autoplace no)
-			(effects
-				(font
-					(size 1.27 1.27)
-				)
-			)
-		)
-		(property "Footprint" "main_pcb:DFrobot"
-			(at 101.346 73.914 0)
-			(hide yes)
-			(show_name no)
-			(do_not_autoplace no)
-			(effects
-				(font
-					(size 1.27 1.27)
-				)
-			)
-		)
-		(property "Datasheet" ""
-			(at 93.98 72.39 0)
-			(hide yes)
-			(show_name no)
-			(do_not_autoplace no)
-			(effects
-				(font
-					(size 1.27 1.27)
-				)
-			)
-		)
-		(property "Description" ""
-			(at 93.98 72.39 0)
-			(hide yes)
-			(show_name no)
-			(do_not_autoplace no)
-			(effects
-				(font
-					(size 1.27 1.27)
-				)
-			)
-		)
-		(pin "3"
-		)
-		(pin "2"
-		)
-		(pin "1"
-		)
-		(pin "4"
-		)
-		(pin "5"
-		)
-		(instances
-			(project "main_pcb"
-				(path "/f7c433f5-979d-4748-9c6b-df3b09da91ad"
-					(reference "U6")
-					(unit 1)
-				)
-			)
-		)
-	)
-	(symbol
 		(lib_id "Device:C_Small")
 		(at 228.6 88.9 270)
@@
 	)
 	(symbol
+		(lib_id "Connector_Generic:Conn_01x02")
+		(at 96.52 67.31 0)
+		(unit 1)
+		(body_style 1)
+		(exclude_from_sim no)
+		(in_bom yes)
+		(on_board yes)
+		(in_pos_files yes)
+		(dnp no)
+		(property "Reference" "J4"
+			(at 96.52 65.024 0)
+			(show_name no)
+			(do_not_autoplace no)
+			(effects
+				(font
+					(size 1.27 1.27)
+				)
+			)
+		)
+		(property "Value" "Pressure_pins"
+			(at 92.202 74.168 0)
+			(show_name no)
+			(do_not_autoplace no)
+			(effects
+				(font
+					(size 1.27 1.27)
+				)
+			)
+		)
+		(property "Footprint" "Connector_PinHeader_2.54mm:PinHeader_1x02_P2.54mm_Vertical"
+			(at 96.52 67.31 0)
+			(hide yes)
+			(show_name no)
+			(do_not_autoplace no)
+			(effects
+				(font
+					(size 1.27 1.27)
+				)
+			)
+		)
+		(property "Datasheet" ""
+			(at 96.52 67.31 0)
+			(hide yes)
+			(show_name no)
+			(do_not_autoplace no)
+			(effects
+				(font
+					(size 1.27 1.27)
+				)
+			)
+		)
+		(property "Description" "Generic connector, single row, 01x02, script generated (kicad-library-utils/schlib/autogen/connector/)"
+			(at 96.52 67.31 0)
+			(hide yes)
+			(show_name no)
+			(do_not_autoplace no)
+			(effects
+				(font
+					(size 1.27 1.27)
+				)
+			)
+		)
+		(pin "1"
+		)
+		(pin "2"
+		)
+		(instances
+			(project "main_pcb"
+				(path "/f7c433f5-979d-4748-9c6b-df3b09da91ad"
+					(reference "J4")
+					(unit 1)
+				)
+			)
+		)
+	)
+	(symbol
 		(lib_id "power:+3.3V")
 		(at 77.47 175.26 180)
@@
 					(unit 1)
 				)
+			)
+		)
+	)
+	(symbol
+		(lib_id "Connector_Generic:Conn_01x03")
+		(at 106.68 68.58 0)
+		(mirror y)
+		(unit 1)
+		(body_style 1)
+		(exclude_from_sim no)
+		(in_bom yes)
+		(on_board yes)
+		(in_pos_files yes)
+		(dnp no)
+		(property "Reference" "J5"
+			(at 107.95 63.754 0)
+			(show_name no)
+			(do_not_autoplace no)
+			(effects
+				(font
+					(size 1.27 1.27)
+				)
+				(justify left)
+			)
+		)
+		(property "Value" "converter_pins"
+			(at 119.38 74.168 0)
+			(show_name no)
+			(do_not_autoplace no)
+			(effects
+				(font
+					(size 1.27 1.27)
+				)
+				(justify left)
+			)
+		)
+		(property "Footprint" "main_pcb:PinHeader_1x03_P2.54mm_Vertical"
+			(at 106.68 68.58 0)
+			(hide yes)
+			(show_name no)
+			(do_not_autoplace no)
+			(effects
+				(font
+					(size 1.27 1.27)
+				)
+			)
+		)
+		(property "Datasheet" ""
+			(at 106.68 68.58 0)
+			(hide yes)
+			(show_name no)
+			(do_not_autoplace no)
+			(effects
+				(font
+					(size 1.27 1.27)
+				)
+			)
+		)
+		(property "Description" "Generic connector, single row, 01x03, script generated (kicad-library-utils/schlib/autogen/connector/)"
+			(at 106.68 68.58 0)
+			(hide yes)
+			(show_name no)
+			(do_not_autoplace no)
+			(effects
+				(font
+					(size 1.27 1.27)
+				)
+			)
+		)
+		(pin "3"
+		)
+		(pin "2"
+		)
+		(pin "1"
+		)
+		(instances
+			(project "main_pcb"
+				(path "/f7c433f5-979d-4748-9c6b-df3b09da91ad"
+					(reference "J5")
+					(unit 1)
+				)
