File: hardware/src/PCB/main_pcb.kicad_sch (KiCad schematic)
At the start: 46 parts, among them J1 Batt, J2 Hall_sensor, J3 Pressure_sensor, J4 Pressure_pins, J5 converter_pins, Q2 BS170, Q4 IRF9530, Q5 IRF9530, Q6 IRF9530, SW1 Button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

Commit message: feature: PCB finished finally AAAAAAAAAAAAAAAAAAAAH
Parts:
- C11, C9: footprint Capacitor_SMD:C_0603_1608Metric -> Capacitor_SMD:C_1206_3216Metric_Pad1.33x1.80mm_HandSolder
- C12, C15, C3, C5, C6, C7, C8: footprint Capacitor_SMD:C_0603_1608Metric -> Capacitor_THT:CP_Radial_Tantal_D5.0mm_P2.50mm
- U5: footprint (none) -> main_pcb:CC1101
Connections:
- net RF_GDO0: now also U2.21 (P1.03_D17_SCK1); no longer U2.23 (P1.07_D19_MOSI1)
- net at R16.2: now also U2.23 (P1.07_D19_MOSI1); no longer U2.21 (P1.03_D17_SCK1)
- net at R17.2: now also U2.11 (P1.15_D10_MOSI); no longer U2.9 (P1.13_D8_SCK)
- net at R15.2: now also U2.9 (P1.13_D8_SCK); no longer U2.11 (P1.15_D10_MOSI)
Other:
- moved on the sheet: R15, R16, R17
Changed lines of the file:
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@@
 	(wire
 		(pts
-			(xy 260.35 135.89) (xy 261.62 135.89)
+			(xy 260.35 140.97) (xy 261.62 140.97)
 		)
 		(stroke
@@
 	(wire
 		(pts
-			(xy 194.31 53.34) (xy 196.85 53.34)
+			(xy 251.46 140.97) (xy 252.73 140.97)
 		)
 		(stroke
@@
 	(wire
 		(pts
-			(xy 193.04 123.19) (xy 203.2 123.19)
+			(xy 194.31 53.34) (xy 196.85 53.34)
 		)
 		(stroke
@@
 	(wire
 		(pts
-			(xy 193.04 130.81) (xy 194.31 130.81)
+			(xy 193.04 123.19) (xy 203.2 123.19)
 		)
 		(stroke
@@
 	(wire
 		(pts
-			(xy 264.16 43.18) (xy 264.16 44.45)
+			(xy 193.04 130.81) (xy 194.31 130.81)
 		)
 		(stroke
@@
 	(wire
 		(pts
-			(xy 137.16 157.48) (xy 137.16 158.75)
+			(xy 264.16 43.18) (xy 264.16 44.45)
 		)
 		(stroke
@@
 	(wire
 		(pts
-			(xy 231.14 87.63) (xy 232.41 87.63)
+			(xy 137.16 157.48) (xy 137.16 158.75)
 		)
 		(stroke
@@
 	(wire
 		(pts
-			(xy 247.65 44.45) (xy 256.54 44.45)
+			(xy 231.14 87.63) (xy 232.41 87.63)
 		)
 		(stroke
@@
 	(wire
 		(pts
-			(xy 128.27 163.83) (xy 129.54 163.83)
+			(xy 247.65 44.45) (xy 256.54 44.45)
 		)
 		(stroke
@@
 	(wire
 		(pts
-			(xy 252.73 127) (xy 251.46 127)
+			(xy 128.27 163.83) (xy 129.54 163.83)
 		)
 		(stroke
@@
 	(wire
 		(pts
-			(xy 251.46 135.89) (xy 252.73 135.89)
-		)
-		(stroke
-			(width 0)
-			(type default)
-		)
-	)
-	(wire
-		(pts
 			(xy 247.65 52.07) (xy 248.92 52.07)
 		)
@@
 	(wire
 		(pts
-			(xy 251.46 140.97) (xy 261.62 140.97)
-		)
-		(stroke
-			(width 0)
-			(type default)
-		)
-	)
-	(wire
-		(pts
 			(xy 201.93 154.94) (xy 203.2 154.94)
 		)
@@
 	(wire
 		(pts
+			(xy 251.46 127) (xy 252.73 127)
+		)
+		(stroke
+			(width 0)
+			(type default)
+		)
+	)
+	(wire
+		(pts
 			(xy 93.98 121.92) (xy 96.52 121.92)
 		)
@@
 	(wire
 		(pts
+			(xy 251.46 119.38) (xy 252.73 119.38)
+		)
+		(stroke
+			(width 0)
+			(type default)
+		)
+	)
+	(wire
+		(pts
 			(xy 88.9 67.31) (xy 90.17 67.31)
 		)
@@
 	(wire
 		(pts
-			(xy 260.35 127) (xy 261.62 127)
+			(xy 260.35 119.38) (xy 261.62 119.38)
 		)
 		(stroke
@@
 	(wire
 		(pts
-			(xy 252.73 119.38) (xy 251.46 119.38)
+			(xy 251.46 135.89) (xy 261.62 135.89)
 		)
 		(stroke
@@
 	(wire
 		(pts
-			(xy 260.35 119.38) (xy 261.62 119.38)
+			(xy 260.35 127) (xy 261.62 127)
 		)
 		(stroke
@@
 	(hierarchical_label "RF_CSN"
 		(shape input)
-		(at 261.62 135.89 0)
+		(at 261.62 140.97 0)
 		(effects
 			(font
@@
 	(hierarchical_label "RF_GDO0"
 		(shape input)
-		(at 261.62 140.97 0)
+		(at 261.62 135.89 0)
 		(effects
 			(font
@@
 	(hierarchical_label "MOSI1"
 		(shape input)
-		(at 261.62 127 0)
+		(at 261.62 119.38 0)
 		(effects
 			(font
@@
 	(hierarchical_label "SCK1"
 		(shape input)
-		(at 261.62 119.38 0)
+		(at 261.62 127 0)
 		(effects
 			(font
@@
 	(symbol
 		(lib_id "Device:R")
-		(at 256.54 135.89 270)
+		(at 256.54 140.97 270)
 		(unit 1)
 		(body_style 1)
@@
 		(dnp no)
 		(property "Reference" "R16"
-			(at 254.508 135.89 90)
+			(at 254.508 140.97 90)
 			(show_name no)
 			(do_not_autoplace no)
@@
 		)
 		(property "Value" "33 Ω"
-			(at 253.746 137.922 90)
+			(at 253.746 143.002 90)
 			(show_name no)
 			(do_not_autoplace no)
@@
 		)
 		(property "Footprint" "main_pcb:R_1206_3216Metric"
-			(at 256.54 134.112 90)
+			(at 256.54 139.192 90)
 			(hide yes)
 			(show_name no)
@@
 		)
 		(property "Datasheet" ""
-			(at 256.54 135.89 0)
+			(at 256.54 140.97 0)
 			(hide yes)
 			(show_name no)
@@
 		)
 		(property "Description" "Resistor"
-			(at 256.54 135.89 0)
+			(at 256.54 140.97 0)
 			(hide yes)
 			(show_name no)
@@
 			)
 		)
-		(property "Footprint" "Capacitor_SMD:C_0603_1608Metric"
+		(property "Footprint" "Capacitor_THT:CP_Radial_Tantal_D5.0mm_P2.50mm"
 			(at 228.6 88.9 0)
 			(hide yes)
@@
 			)
 		)
-		(property "Footprint" "Capacitor_SMD:C_0603_1608Metric"
+		(property "Footprint" "Capacitor_THT:CP_Radial_Tantal_D5.0mm_P2.50mm"
 			(at 45.72 36.83 0)
 			(hide yes)
@@
 			)
 		)
-		(property "Footprint" "Capacitor_SMD:C_0603_1608Metric"
+		(property "Footprint" "Capacitor_THT:CP_Radial_Tantal_D5.0mm_P2.50mm"
 			(at 255.27 114.3 0)
 			(hide yes)
@@
 			)
 		)
-		(property "Footprint" "Capacitor_SMD:C_0603_1608Metric"
+		(property "Footprint" "Capacitor_THT:CP_Radial_Tantal_D5.0mm_P2.50mm"
 			(at 44.45 67.31 0)
 			(hide yes)
@@
 			)
 		)
-		(property "Footprint" "Capacitor_SMD:C_0603_1608Metric"
+		(property "Footprint" "Capacitor_SMD:C_1206_3216Metric_Pad1.33x1.80mm_HandSolder"
 			(at 96.52 119.38 0)
 			(hide yes)
@@
 	(symbol
 		(lib_id "Device:R")
-		(at 256.54 127 270)
+		(at 256.54 119.38 270)
 		(unit 1)
 		(body_style 1)
@@
 		(dnp no)
 		(property "Reference" "R17"
-			(at 254.508 127 90)
+			(at 254.508 119.38 90)
 			(show_name no)
 			(do_not_autoplace no)
@@
 		)
 		(property "Value" "33 Ω"
-			(at 254.254 124.968 90)
+			(at 254 121.412 90)
 			(show_name no)
 			(do_not_autoplace no)
@@
 		)
 		(property "Footprint" "main_pcb:R_1206_3216Metric"
-			(at 256.54 125.222 90)
+			(at 256.54 117.602 90)
 			(hide yes)
 			(show_name no)
@@
 		)
 		(property "Datasheet" ""
-			(at 256.54 127 0)
+			(at 256.54 119.38 0)
 			(hide yes)
 			(show_name no)
@@
 		)
 		(property "Description" "Resistor"
-			(at 256.54 127 0)
+			(at 256.54 119.38 0)
 			(hide yes)
 			(show_name no)
@@
 			)
 		)
-		(property "Footprint" "Capacitor_SMD:C_0603_1608Metric"
+		(property "Footprint" "Capacitor_THT:CP_Radial_Tantal_D5.0mm_P2.50mm"
 			(at 100.33 36.83 0)
 			(hide yes)
@@
 			)
 		)
-		(property "Footprint" "Capacitor_SMD:C_0603_1608Metric"
+		(property "Footprint" "Capacitor_SMD:C_1206_3216Metric_Pad1.33x1.80mm_HandSolder"
 			(at 196.85 50.8 0)
 			(hide yes)
@@
 			)
 		)
-		(property "Footprint" "Capacitor_SMD:C_0603_1608Metric"
+		(property "Footprint" "Capacitor_THT:CP_Radial_Tantal_D5.0mm_P2.50mm"
 			(at 260.35 44.45 0)
 			(hide yes)
@@
 	(symbol
 		(lib_id "Device:R")
-		(at 256.54 119.38 270)
+		(at 256.54 127 270)
 		(unit 1)
 		(body_style 1)
@@
 		(dnp no)
 		(property "Reference" "R15"
-			(at 254.508 119.38 90)
+			(at 254.508 127 90)
 			(show_name no)
 			(do_not_autoplace no)
@@
 		)
 		(property "Value" "33 Ω"
-			(at 254 121.666 90)
+			(at 254 124.968 90)
 			(show_name no)
 			(do_not_autoplace no)
@@
 		)
 		(property "Footprint" "main_pcb:R_1206_3216Metric"
-			(at 256.54 117.602 90)
+			(at 256.54 125.222 90)
 			(hide yes)
 			(show_name no)
@@
 		)
 		(property "Datasheet" ""
-			(at 256.54 119.38 0)
+			(at 256.54 127 0)
 			(hide yes)
 			(show_name no)
@@
 		)
 		(property "Description" "Resistor"
-			(at 256.54 119.38 0)
+			(at 256.54 127 0)
 			(hide yes)
 			(show_name no)
@@
 		)
 		(property "Field5" ""
-			(at 256.54 119.38 90)
+			(at 256.54 127 90)
 			(hide yes)
 			(show_name no)
@@
 		)
 		(property "Field6" ""
-			(at 256.54 119.38 90)
+			(at 256.54 127 90)
 			(hide yes)
 			(show_name no)
@@
 		)
 		(property "Field7" ""
-			(at 256.54 119.38 90)
+			(at 256.54 127 90)
 			(hide yes)
 			(show_name no)
@@
 			)
 		)
-		(property "Footprint" "Capacitor_SMD:C_0603_1608Metric"
+		(property "Footprint" "Capacitor_THT:CP_Radial_Tantal_D5.0mm_P2.50mm"
 			(at 114.3 67.31 0)
 			(hide yes)
@@
 			)
 		)
-		(property "Footprint" ""
+		(property "Footprint" "main_pcb:CC1101"
 			(at 251.46 58.42 0)
 			(hide yes)
