File: hardware/src/PCB/main_pcb.kicad_pcb (KiCad board)
At the start: 2 copper layers, 11 parts, among them J1 Servo_motor, J2 Sen057_pressure_sensor, J3 Hall_effect_sensor, J4 Jack plug, SW1 SPDT_Slide_SMD_6.7x2.6mm, SW2 telemetry_btn, U1 XIAO-nRF52840-Plus-SMD, U2 5V_booster, U5 Openlog_SDcard, U6 Radio_module

Commit message: feature: PCB  advancement
Parts:
- removed J2: Sen057_pressure_sensor, Connector_PinHeader_2.54mm:PinHeader_1x03_P2.54mm_Vertical
- removed J3: Hall_effect_sensor, Connector_PinHeader_2.54mm:PinHeader_1x03_P2.54mm_Vertical
- removed J4: Jack plug, Connector_PinHeader_2.54mm:PinHeader_1x02_P2.54mm_Horizontal
- removed SW2: telemetry_btn, craby's_library:SW_BUTT-2
- removed U1: XIAO-nRF52840-Plus-SMD, XIAO_Series_Footprints:XIAO-nRF52840-Plus-SMD
- removed U5: Openlog_SDcard, craby's_library:Openlog_SDreader
- removed U6: Radio_module, craby's_library:Ebyte_radio_module
- BZ1: value Buzzer_info -> Buzzer; footprint Buzzer_Beeper:Buzzer_12x9.5RM7.6 -> Buzzer_Beeper:MagneticBuzzer_ProSignal_ABT-410-RC
- J1: value Servo_motor -> Conn_01x03; footprint Connector_PinHeader_2.54mm:PinHeader_1x03_P2.54mm_Vertical -> main_pcb:PinHeader_1x03_P2.54mm_Vertical
- SW1: value SPDT_Slide_SMD_6.7x2.6mm -> Button; footprint Button_Switch_SMD:SW_SPDT_CK_JS102011SAQN -> Button_Switch_SMD:SW_SPST_B3U-1000P
- U2: value 5V_booster -> XIAO-nRF52840-Plus-SMD; footprint craby's_library:5V_booster -> main_pcb:XIAO-nRF52840-Plus-SMD
- moved BZ1 50.7 mm to (143.2, 101.0)
- moved U2 41.1 mm to (150.9, 81.8), turned to 0 degrees
- moved J1 36.7 mm to (157.9, 96.4), turned to 0 degrees
- moved SW1 26.9 mm to (158.5, 105.9), turned to 0 degrees
Connections:
- BZ1 pad 2: GND -> unconnected-(BZ1---Pad2)
- J1 pad 2: +5V -> unconnected-(J1-Pin_2-Pad2)
- J1 pad 3: GND -> unconnected-(J1-Pin_3-Pad3)
- SW1 pad 1: +5V -> Net-(SW1-A-Pad1)
- SW1 pad 2: Net-(U1-VBAT) -> Net-(SW1-A-Pad1)

Commit message: feature: PCB advancement
Parts:
- added C1: 2.2µF - céramique, Capacitor_SMD:C_0603_1608Metric, F.Cu at (97.5, 105.0)
- added C10: 10 µF - céramique, Capacitor_SMD:C_0603_1608Metric, F.Cu at (246.2, 89.0)
- added C11: 100 nF - céramique, Capacitor_SMD:C_0603_1608Metric, F.Cu at (246.2, 91.5)
- added C12: 100 nF - céramique, Capacitor_SMD:C_0603_1608Metric, F.Cu at (246.2, 94.0)
- added C13: 10 µF - céramique, Capacitor_SMD:C_0603_1608Metric, F.Cu at (246.2, 96.5)
- added C14: 10 µF - céramique, Capacitor_SMD:C_0603_1608Metric, F.Cu at (250.2, 84.0)
- added C15: 100 nF - céramique, Capacitor_SMD:C_0603_1608Metric, F.Cu at (250.2, 86.5)
- added C16: 100nF - céramique, Capacitor_SMD:C_0603_1608Metric, F.Cu at (113.8, 88.0)
- added C2: 470 µF - électrolytique, Capacitor_THT:CP_Radial_D10.0mm_P5.00mm, F.Cu at (91.3, 102.5)
- added C3: 2.2 µF - céramique, Capacitor_SMD:C_0603_1608Metric, F.Cu at (113.3, 115.1)
- added C4: 10 µF - céramique, Capacitor_SMD:C_0603_1608Metric, F.Cu at (242.2, 89.0)
- added C5: 100 nF - céramique, Capacitor_SMD:C_0603_1608Metric, F.Cu at (242.2, 91.5)
- added C6: 100 nF - céramique, Capacitor_SMD:C_0603_1608Metric, F.Cu at (242.2, 94.0)
- added C7: 100 nF - céramique, Capacitor_SMD:C_0603_1608Metric, F.Cu at (242.2, 96.5)
- added C8: 100 nF - céramique, Capacitor_SMD:C_0603_1608Metric, F.Cu at (246.2, 84.0)
- added C9: 100 nF - céramique, Capacitor_SMD:C_0603_1608Metric, F.Cu at (246.2, 86.5)
- added D1: SS14, Diode_SMD:D_SMA, F.Cu at (82.3, 104.0)
- added D2: 1N4148W, Diode_SMD:D_SOD-123, F.Cu at (91.5, 89.0)
- added J2: Hall_sensor, main_pcb:PinHeader_1x03_P2.54mm_Vertical, F.Cu at (258.4, 91.8)
- added J3: Pressure_sensor, Connector_PinHeader_2.54mm:PinHeader_1x02_P2.54mm_Vertical, F.Cu at (257.4, 77.3)
- added Q1: BSS84, Package_TO_SOT_SMD:SOT-23, F.Cu at (255.3, 47.6)
- added Q2: BSS138, Package_TO_SOT_SMD:SOT-23, F.Cu at (255.3, 52.1)
- added Q3: BSS84, Package_TO_SOT_SMD:SOT-23, F.Cu at (255.3, 56.5)
- added Q4: BSS84, Package_TO_SOT_SMD:SOT-23, F.Cu at (255.3, 61.0)
- added R1: 100Ω, Resistor_SMD:R_0201_0603Metric, F.Cu at (115.6, 94.4)
- added R10: 100k Ω, Resistor_SMD:R_0201_0603Metric, F.Cu at (261.4, 58.5)
- added R11: 100 Ω, Resistor_SMD:R_0201_0603Metric, F.Cu at (110.5, 94.4)
- added R12: 100Ω, Resistor_SMD:R_0201_0603Metric, F.Cu at (101.6, 94.3)
- added R13: 100Ω, Resistor_SMD:R_0201_0603Metric, F.Cu at (101.6, 115.1)
- added R14: 100k Ω, Resistor_SMD:R_0201_0603Metric, F.Cu at (261.4, 65.5)
- added R15: 33Ω, Resistor_SMD:R_0201_0603Metric, F.Cu at (109.3, 115.1)
- added R16: 33Ω, Resistor_SMD:R_0201_0603Metric, F.Cu at (102.9, 115.1)
- added R17: 33 Ω, Resistor_SMD:R_0201_0603Metric, F.Cu at (104.2, 115.1)
- added R18: 100k Ω, Resistor_SMD:R_0201_0603Metric, F.Cu at (263.9, 60.3)
- added R19: 100k Ω, Resistor_SMD:R_0201_0603Metric, F.Cu at (263.9, 62.0)
- added R2: 10k Ω, Resistor_SMD:R_0201_0603Metric, F.Cu at (258.9, 58.5)
- added R20: 100k Ω, Resistor_SMD:R_0201_0603Metric, F.Cu at (263.9, 63.8)
- added R3: 10k Ω, Resistor_SMD:R_0201_0603Metric, F.Cu at (258.9, 60.3)
- added R4: 10k Ω, Resistor_SMD:R_0201_0603Metric, F.Cu at (258.9, 62.0)
- added R5: 100 Ω, Resistor_SMD:R_0201_0603Metric, F.Cu at (114.3, 94.4)
- added R6: 1kΩ, Resistor_SMD:R_0201_0603Metric, F.Cu at (111.6, 88.0)
- added R7: 100k Ω, Resistor_SMD:R_0201_0603Metric, F.Cu at (258.9, 67.3)
- added R8: 100 Ω, Resistor_SMD:R_0201_0603Metric, F.Cu at (113.1, 94.4)
- added SW2: Button, Button_Switch_SMD:SW_SPST_B3U-1000P, F.Cu at (263.6, 78.5)
- added U1: ~, main_pcb:Adafruit_TPS61040_5644, F.Cu at (227.6, 92.2)
- added U3: ~, main_pcb:BME280, F.Cu at (245.8, 76.6)
- added U4: ~, main_pcb:OpenLog, F.Cu at (233.8, 78.6)
- added U6: ~, main_pcb:DFrobot, F.Cu at (236.3, 57.9)
- J1: value Conn_01x03 -> Batt; footprint main_pcb:PinHeader_1x03_P2.54mm_Vertical -> PCM_SparkFun-Connector:JST_1x02_P2.0mm_Horizontal_SMD; moved to B.Cu
- moved SW1 110.8 mm to (264.0, 72.0)
- moved J1 83.6 mm to (74.8, 105.3), turned to -90 degrees
- moved BZ1 59.8 mm to (84.0, 92.1), turned to 90 degrees
- moved U2 47.6 mm to (109.2, 104.7)
Connections:
- BZ1 pad 1: unconnected-(BZ1-+-Pad1) -> +3.3V
- BZ1 pad 2: unconnected-(BZ1---Pad2) -> GND
- J1 pad 1: unconnected-(J1-Pin_1-Pad1) -> +3.3V
- J1 pad 2: unconnected-(J1-Pin_2-Pad2) -> GND
- SW1 pad 1: Net-(SW1-A-Pad1) -> /Button
- SW1 pad 2: Net-(SW1-A-Pad1) -> /Button
- U2 pad 1: unconnected-(U2-P0.02_A0_D0-Pad1) -> /Button
- U2 pad 10: unconnected-(U2-P1.14_D9_MISO-Pad10) -> /MISO1
- U2 pad 11: unconnected-(U2-P1.15_D10_MOSI-Pad11) -> Net-(U2-P1.15_D10_MOSI)
- U2 pad 14: +5V -> unconnected-(U2-VBUS-Pad14)
- U2 pad 15: unconnected-(U2-P0.15_D11_I2S_SD-Pad15) -> Net-(U2-P0.15_D11_I2S_SD)
- U2 pad 16: unconnected-(U2-P0.19_D12_I2S_SCK-Pad16) -> Net-(U2-P0.19_D12_I2S_SCK)
- U2 pad 17: unconnected-(U2-P1.01_D13_I2S_WS-Pad17) -> Net-(U2-P1.01_D13_I2S_WS)
- U2 pad 2: unconnected-(U2-P0.03_A1_D1-Pad2) -> Net-(U2-P0.03_A1_D1)
- U2 pad 20: unconnected-(U2-P0.31_D16_BAT-Pad20) -> Net-(D1-K)
- U2 pad 21: unconnected-(U2-P1.03_D17_SCK1-Pad21) -> Net-(U2-P1.03_D17_SCK1)
- U2 pad 23: unconnected-(U2-P1.07_D19_MOSI1-Pad23) -> /RF_GDO0
- U2 pad 26: unconnected-(U2-REST-Pad26) -> /Rst_btn
- U2 pad 27: GND -> unconnected-(U2-GND-Pad27)
- U2 pad 3: unconnected-(U2-P0.28_A2_D2-Pad3) -> Net-(U2-P0.28_A2_D2)
- U2 pad 4: unconnected-(U2-P0.29_A3_D3-Pad4) -> /Hall
- U2 pad 5: unconnected-(U2-P0.04_A4_D4_SDA-Pad5) -> /SDA1
- U2 pad 6: unconnected-(U2-P0.05_A5_D5_SCL-Pad6) -> /SCL1
- U2 pad 7: unconnected-(U2-P1.11_D6_TX-Pad7) -> Net-(U2-P1.11_D6_TX)
- U2 pad 8: unconnected-(U2-P1.12_D7_RX-Pad8) -> Net-(U2-P1.12_D7_RX)
- U2 pad 9: unconnected-(U2-P1.13_D8_SCK-Pad9) -> Net-(U2-P1.13_D8_SCK)
Routing:
- net Net-(D1-K): track 0.00 -> 21.9 mm
- net GND: track 0.00 -> 13.1 mm
Other:
- board outline added: 80 x 80 mm

Commit message: feature: PCB advancement
Parts:
- removed C1: 2.2µF - céramique, Capacitor_SMD:C_0603_1608Metric
- removed Q1, Q3: BSS84, Package_TO_SOT_SMD:SOT-23
- added C17: 220 µF - électrolytique, Capacitor_THT:CP_Radial_D10.0mm_P5.00mm, F.Cu at (238.7, 81.4)
- added Q5: IRF9530, main_pcb:TRANS_IRF9530, F.Cu at (235.9, 111.1)
- added Q6: IRF9530, main_pcb:TRANS_IRF9530, F.Cu at (235.9, 117.1)
- C16: value 100nF - céramique -> 100 nF - céramique
- C2: value 470 µF - électrolytique -> 47 µF - électrolytique
- C3: value 2.2 µF - céramique -> 2.2 µF - céramique
- D1: value SS14 -> 1N5819; footprint Diode_SMD:D_SMA -> main_pcb:DIOAD1036W78L470D235
- D2: value 1N4148W -> fr107; footprint Diode_SMD:D_SOD-123 -> main_pcb:DIOAD1036W78L470D235
- J1: footprint PCM_SparkFun-Connector:JST_1x02_P2.0mm_Horizontal_SMD -> Connector_PinHeader_1.00mm:PinHeader_1x02_P1.00mm_Horizontal; moved to F.Cu
- Q2: value BSS138 -> BS170; footprint Package_TO_SOT_SMD:SOT-23 -> main_pcb:TO92
- Q4: value BSS84 -> IRF9530; footprint Package_TO_SOT_SMD:SOT-23 -> main_pcb:TRANS_IRF9530
- R1, R12, R13: value 100Ω -> 100 Ω; footprint Resistor_SMD:R_0201_0603Metric -> main_pcb:R_1206_3216Metric
- R10, R11, R14, R17, R18, R19, R2, R20, R3, R4, R5, R7, R8: footprint Resistor_SMD:R_0201_0603Metric -> main_pcb:R_1206_3216Metric
- R15, R16: value 33Ω -> 33 Ω; footprint Resistor_SMD:R_0201_0603Metric -> main_pcb:R_1206_3216Metric
- R6: value 1kΩ -> 1k Ω; footprint Resistor_SMD:R_0201_0603Metric -> main_pcb:R_1206_3216Metric
- moved D1 156.1 mm to (237.9, 91.0), turned to 0 degrees
- moved C2 151.0 mm to (238.7, 69.8), turned to 0 degrees
- moved D2 146.5 mm to (237.9, 95.0), turned to 0 degrees
- moved BZ1 136.3 mm to (219.4, 108.1), turned to 0 degrees
- moved J1 118.3 mm to (192.1, 120.9), turned to 0 degrees
- moved R16 112.8 mm to (213.0, 90.8), turned to 0 degrees
- moved R17 110.8 mm to (213.0, 94.1), turned to 0 degrees
- moved R13 106.4 mm to (207.4, 104.0), turned to 0 degrees
- moved R12 106.0 mm to (207.4, 100.7), turned to 0 degrees
- moved R15 98.2 mm to (207.4, 110.6), turned to 0 degrees
- moved R11 97.0 mm to (207.4, 97.4), turned to 0 degrees
- moved R8 94.4 mm to (207.4, 90.8), turned to 0 degrees
- moved R6 92.2 mm to (201.8, 107.3), turned to 0 degrees
- moved U2 88.2 mm to (191.0, 137.6)
- moved R5 88.0 mm to (201.8, 104.0), turned to 0 degrees
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Routing:
- net Net-(D1-K): track 21.9 -> 0.00 mm
- net GND: track 13.1 -> 0.00 mm
- added copper zone on F.Cu, net GND

Commit message: feature: PCB advancement
Parts:
- removed C17: 220 µF - électrolytique, Capacitor_THT:CP_Radial_D10.0mm_P5.00mm
- removed Q4: IRF9530, main_pcb:TRANS_IRF9530
- removed R18, R20: 100k Ω, main_pcb:R_1206_3216Metric
- removed R3, R4: 10k Ω, main_pcb:R_1206_3216Metric
- BZ1, C2, D1, D2, J2, J3, Q2, Q5, Q6, U1, U4: moved to B.Cu
- J1: footprint Connector_PinHeader_1.00mm:PinHeader_1x02_P1.00mm_Horizontal -> Connector_PinHeader_2.54mm:PinHeader_1x02_P2.54mm_Horizontal; moved to B.Cu
- moved D1 150.1 mm to (88.4, 104.3)
- moved C2 143.0 mm to (99.8, 104.2), turned to -90 degrees
- moved U3 134.3 mm to (87.6, 84.2), turned to 90 degrees
- moved J2 134.3 mm to (113.2, 80.4), turned to -90 degrees
- moved Q6 131.8 mm to (104.2, 120.8), turned to 90 degrees
- moved Q5 125.5 mm to (115.6, 75.5), turned to 180 degrees
- moved U6 120.6 mm to (78.9, 44.0)
- moved J1 113.0 mm to (80.3, 104.7), turned to 180 degrees
- moved R10 107.7 mm to (104.9, 127.3)
- moved R16 105.4 mm to (111.2, 117.8), turned to 90 degrees
- moved D2 105.3 mm to (133.4, 107.9), turned to -90 degrees
- moved R14 103.6 mm to (109.1, 74.6), turned to -90 degrees
- moved J3 103.5 mm to (140.6, 98.6), turned to 90 degrees
- moved R17 102.3 mm to (113.5, 117.8), turned to 90 degrees
- moved R13 99.5 mm to (108.8, 117.8), turned to 90 degrees
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Connections:
- D1 pad C: (no net) -> +3.3V
- D2 pad A: (no net) -> +3.3V
- D2 pad C: (no net) -> GND
- Q2 pad 2: GND -> Net-(Q2-S)
- Q2 pad 3: Net-(Q2-D) -> GND
- R1 pad 1: GND -> +3.3V
- R19 pad 1: GND -> /MOSFET2
- R5 pad 1: +3.3V -> /MOSFET2
- SW1 pad 2: /Button -> GND
- U2 pad 28: (no net) -> +3.3V
- U2 pad 29: (no net) -> GND
Routing:
- net +3.3V: track 0.00 -> 44.0 mm
- net GND: track 0.00 -> 33.3 mm
- net Net-(D1-K): track 0.00 -> 18.8 mm
- net /SD_RX: track 0.00 -> 18.0 mm
- net /MOSFET2: track 0.00 -> 8.34 mm
- net /Button: track 0.00 -> 5.13 mm
- net +12V: track 0.00 -> 4.52 mm
- net /Hall: track 0.00 -> 4.11 mm
- net Net-(U2-P0.15_D11_I2S_SD): track 0.00 -> 3.80 mm
- net Net-(U2-P0.03_A1_D1): track 0.00 -> 3.00 mm
- net Net-(U2-P1.13_D8_SCK): track 0.00 -> 2.73 mm
- net Net-(U2-P1.12_D7_RX): track 0.00 -> 2.72 mm
- net Net-(U2-P1.01_D13_I2S_WS): track 0.00 -> 2.57 mm
- net Net-(U2-P0.28_A2_D2): track 0.00 -> 2.55 mm
- net Net-(U2-P1.11_D6_TX): track 0.00 -> 2.38 mm
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- removed copper zone on F.Cu, net GND

Commit message: feature: PCB advancement
Parts:
- removed SW2: Button, Button_Switch_SMD:SW_SPST_B3U-1000P
- added C17: 220 µF - électrolytique, Capacitor_THT:CP_Radial_D8.0mm_P3.50mm, B.Cu at (84.8, 99.1)
- added Q4: IRF9530, main_pcb:TRANS_IRF9530, B.Cu at (121.4, 74.1)
- added R18: 100k Ω, main_pcb:R_1206_3216Metric, F.Cu at (120.3, 76.7)
- J1: footprint Connector_PinHeader_2.54mm:PinHeader_1x02_P2.54mm_Horizontal -> Connector_PinHeader_2.54mm:PinHeader_1x02_P2.54mm_Vertical; moved to F.Cu
- J2, J3: moved to F.Cu
- U3: moved to B.Cu
- moved U6 162.2 mm to (232.1, 97.5)
- moved C9 73.8 mm to (232.1, 76.0)
- moved C10 73.8 mm to (232.1, 78.5)
- moved C11 73.8 mm to (232.1, 81.1)
- moved C12 73.8 mm to (232.1, 83.6)
- moved C8 73.8 mm to (232.1, 73.5)
- moved C13 73.8 mm to (236.1, 73.5)
- moved C14 73.8 mm to (236.1, 76.0)
- moved C15 73.8 mm to (236.1, 78.5)
- moved C16 73.8 mm to (236.1, 81.1)
- moved C3 73.8 mm to (228.1, 73.5)
- moved C4 73.8 mm to (228.1, 76.0)
- moved C5 73.8 mm to (228.1, 78.5)
- moved C6 73.8 mm to (228.1, 81.1)
- moved C7 73.8 mm to (228.1, 83.6)
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Connections:
- C11 pad 1: +3.3V -> /Transistor+
- C2 pad 1: Net-(D1-K) -> +3.3V
- D1 pad A: (no net) -> +3.3V
- D2 pad A: +3.3V -> (no net)
- D2 pad C: GND -> (no net)
- Q2 pad 3: GND -> /Transistor+
- R1 pad 1: +3.3V -> /Transistor+
- R19 pad 1: /MOSFET2 -> GND
- R19 pad 2: GND -> /Transistor+
- R5 pad 1: /MOSFET2 -> +3.3V
- R7 pad 2: GND -> /Transistor+
- U1 pad 1: +3.3V -> /Transistor+
- U2 pad 20: Net-(D1-K) -> +3.3V
Routing:
- net +3.3V: track 44.0 -> 91.3 mm, vias 0 -> 1
- net /Hall: track 4.11 -> 39.0 mm
- net /Transistor+: track 0.00 -> 33.4 mm
- net /MOSFET2: track 8.34 -> 34.6 mm
- net /SDA1: track 0.00 -> 21.7 mm
- net GND: track 33.3 -> 11.8 mm
- net Net-(D1-K): track 18.8 -> 0.00 mm
- net /SCL1: track 0.00 -> 17.5 mm
- net /SD_RX: track 18.0 -> 35.1 mm
- net /SD_TX: track 0.00 -> 8.82 mm
- net Net-(Q2-S): track 0.00 -> 5.76 mm
- net +12V: track 4.52 -> 0.08 mm
- net /MOSFET3: track 0.00 -> 4.09 mm, vias 0 -> 1
- net /PressureA: track 0.00 -> 1.82 mm, vias 0 -> 1
- added copper zone on F.Cu, net GND
Other:
- board outline removed
- board text added: "CC1101"

Commit message: feature: PCB advancement
Parts:
- removed U6: ~, main_pcb:DFrobot
- added J4: Pressure_pins, Connector_PinHeader_2.54mm:PinHeader_1x02_P2.54mm_Vertical, B.Cu at (133.2, 92.8)
- added J5: converter_pins, main_pcb:PinHeader_1x03_P2.54mm_Vertical, B.Cu at (123.5, 119.5)
- moved R14 25.9 mm to (111.3, 73.2)
- moved Q5 19.4 mm to (108.8, 74.3)
- moved J2 19.4 mm to (103.7, 81.9)
- moved R2 19.4 mm to (100.7, 78.4)
- moved BZ1 8.69 mm to (138.4, 108.1), turned to -90 degrees
- moved J3 6.45 mm to (135.7, 99.0)
- moved U3 6.40 mm to (91.6, 82.4)
- moved D2 1.82 mm to (130.8, 111.7), turned to 90 degrees
Connections:
- D2 pad A: (no net) -> +3.3V
- D2 pad C: (no net) -> GND
- Q2 pad 3: /Transistor+ -> Net-(Q2-S)
- Q4 pad 3: /Transistor+ -> +3.3V
- Q5 pad 1: /MOSFET2 -> +3.3V
- Q5 pad 3: +3.3V -> /MOSFET2
- Q6 pad 1: /MOSFET3 -> +3.3V
- Q6 pad 3: +3.3V -> /MOSFET3
- R10 pad 1: /MOSFET3 -> +3.3V
- R10 pad 2: +3.3V -> /MOSFET3
- R14 pad 1: /MOSFET2 -> +3.3V
- R14 pad 2: +3.3V -> /MOSFET2
- SW1 pad 2: GND -> /Button
- U1 pad 1: /Transistor+ -> +3.3V
Routing:
- net +3.3V: track 91.3 -> 230.1 mm
- net /Hall: track 39.0 -> 20.0 mm
- net /Transistor+: track 33.4 -> 15.9 mm
- net /MOSFET2: track 34.6 -> 17.8 mm
- net /MISO1: track 0.00 -> 14.8 mm
- net /RF_GDO0: track 0.00 -> 13.9 mm
- net /RF_CSN: track 0.00 -> 10.7 mm
- net /MOSI1: track 0.00 -> 9.96 mm
- net /SCK1: track 0.00 -> 9.05 mm
- net GND: track 11.8 -> 3.20 mm
- net +12V: track 0.08 -> 8.44 mm
- net /SCL1: track 17.5 -> 23.9 mm
- net /SDA1: track 21.7 -> 28.1 mm
- net Net-(Q2-S): track 5.76 -> 7.00 mm
- net /MOSFET3: track 4.09 -> 5.12 mm
Other:
- board outline added: 80 x 80 mm

Commit message: feature: PCB finished finally AAAAAAAAAAAAAAAAAAAAH
Parts:
- removed C10, C13, C14, C4: 10 µF - céramique, Capacitor_SMD:C_0603_1608Metric
- removed C16: 100 nF - céramique, Capacitor_SMD:C_0603_1608Metric
- removed C3: 2.2 µF - céramique, Capacitor_SMD:C_0603_1608Metric
- added G***: LOGO, main_pcb:y2k-img, F.Cu at (101.7, 133.6)
- added G***: LOGO, main_pcb:Saturn-img, F.Cu at (95.9, 136.5)
- added U5: ~, main_pcb:CC1101, B.Cu at (127.5, 139.4)
- C11, C9: footprint Capacitor_SMD:C_0603_1608Metric -> Capacitor_SMD:C_1206_3216Metric_Pad1.33x1.80mm_HandSolder
- C12, C15, C5, C6, C7, C8: footprint Capacitor_SMD:C_0603_1608Metric -> Capacitor_THT:CP_Radial_Tantal_D5.0mm_P2.50mm; moved to B.Cu
- moved C9 145.0 mm to (93.0, 116.8), turned to -90 degrees
- moved C7 132.7 mm to (95.5, 88.6), turned to 180 degrees
- moved C8 131.2 mm to (101.0, 75.2), turned to 90 degrees
- moved C15 120.8 mm to (123.5, 122.4), turned to 180 degrees
- moved C12 117.5 mm to (117.8, 110.7), turned to 180 degrees
- moved C11 99.9 mm to (132.2, 84.5)
- moved C5 95.2 mm to (135.8, 101.8)
- moved C6 88.6 mm to (144.7, 111.1), turned to -90 degrees
- moved J3 2.50 mm to (138.2, 99.0)
- moved J4 2.50 mm to (135.8, 92.7)
- moved R19 2.44 mm to (117.8, 82.9), turned to 0 degrees
- moved BZ1 1.46 mm to (137.4, 109.2)
- moved D2 1.46 mm to (129.7, 112.7)
- turned Q4 to 180 degrees
Connections:
- C11 pad 1: /Transistor+ -> +3.3V
- Q2 pad 3: Net-(Q2-S) -> /Transistor+
- Q4 pad 1: Net-(Q2-S) -> +3.3V
- Q4 pad 3: +3.3V -> /Transistor+
- Q5 pad 1: +3.3V -> /MOSFET2
- Q5 pad 3: /MOSFET2 -> +3.3V
- Q6 pad 1: +3.3V -> /MOSFET3
- Q6 pad 3: /MOSFET3 -> +3.3V
- R1 pad 1: /Transistor+ -> Net-(Q2-S)
- R10 pad 1: +3.3V -> /MOSFET3
- R10 pad 2: /MOSFET3 -> +3.3V
- R14 pad 1: +3.3V -> /MOSFET2
- R14 pad 2: /MOSFET2 -> +3.3V
- R15 pad 1: /SCK1 -> /MOSI1
- R16 pad 1: /RF_CSN -> /RF_GDO0
- R17 pad 1: /MOSI1 -> /SCK1
- R18 pad 1: Net-(Q2-S) -> /Transistor+
- R19 pad 2: /Transistor+ -> Net-(Q2-S)
- R7 pad 2: /Transistor+ -> GND
- SW1 pad 2: /Button -> GND
- U2 pad 20: +3.3V -> Net-(D1-K)
- U2 pad 23: /RF_GDO0 -> /RF_CSN
Routing:
- net +3.3V: track 230.1 -> 309.4 mm, vias 1 -> 2
- net /PressureA: track 1.82 -> 39.2 mm, vias 1 -> 2
- net GND: track 3.20 -> 39.0 mm, vias 0 -> 3
- net /MOSFET3: track 5.12 -> 36.8 mm
- net /RF_GDO0: track 13.9 -> 45.2 mm
- net /SCK1: track 9.05 -> 40.0 mm
- net /MISO1: track 14.8 -> 39.1 mm
- net /RF_CSN: track 10.7 -> 28.9 mm, vias 0 -> 2
- net /MOSI1: track 9.96 -> 24.4 mm
- net +12V: track 8.44 -> 12.4 mm
- net /Transistor+: track 15.9 -> 17.8 mm
Other:
- board text added: "If I smoke, don't panic. Just blame the designer. He's bad"
- board text removed: "CC1101"
